File: vgc-zero.kicad_sch (KiCad schematic)
At the start: 25 parts, among them J1 Conn_01x06_Pin, J2 Conn_01x06_Pin, J3 Conn_01x06_Pin, SW1 SW_Push, SW10 SW_Push, SW11 SW_SPDT, SW2 SW_Push, SW3 SW_Push, SW4 SW_Push, SW5 SW_Push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

Commit message: major improvements
Parts:
- removed H1, H2, H3, H4: MountingHole_Pad, MountingHole:MountingHole_2.2mm_M2_Pad, symbol Mechanical:MountingHole_Pad
- added DISP1: DISPLAY, vgc-zero-footprints:SSD1351_OLED_128x128_WAVESHARE, symbol vgc-zero-symbols:SSD1351_OLED_128x128_WAVESHARE
- Buzz1: renamed from LS1; value Speaker -> Buzzer; symbol Device:Speaker -> Device:Buzzer
- DISP1_CONN1: renamed from OLED1; value DISP1 -> DISPLAY_CONNECTOR; symbol vgc-zero-symbols:SSD1351_OLED_128x128_WAVESHARE -> Connector:Conn_01x07_Socket
Connections:
- net GND: now also Buzz1.2 (-), DISP1.1 (GND); no longer Buzz1.1
- net DISP_DIN: now reaches DISP1_CONN1.3 (Pin_3), MCU1.25 (GPIO19)
- net DISP_CLK: now reaches DISP1_CONN1.4 (Pin_4), MCU1.24 (GPIO18)
- net DISP_CS: now reaches DISP1_CONN1.5 (Pin_5), MCU1.22 (GPIO17)
- net DISP_DC: now reaches DISP1_CONN1.6 (Pin_6), MCU1.27 (GPIO21)
- net DISP_RST: now reaches DISP1_CONN1.7 (Pin_7), MCU1.26 (GPIO20)
- net at MCU1.29 (GPIO22): now also Buzz1.1 (+); no longer Buzz1.2
Other:
- moved on the sheet: H5, H6
