File: vgc-zero.kicad_pcb (KiCad board)
At the start: 2 copper layers, 50 x 90 mm, 24 parts, among them J1 Conn_01x06_Pin, J2 Conn_01x06_Pin, J3 Conn_01x06_Pin, SW1 SW_Push, SW10 SW_Push, SW11 SW_SPDT, SW2 SW_Push, SW3 SW_Push, SW4 SW_Push, SW5 SW_Push, SW6 SW_Push, SW7 SW_Push, SW8 SW_Push, SW9 SW_Push

Commit message: new version changes
Parts:
- removed Buzz1: Buzzer, Buzzer_Beeper:Buzzer_12x9.5RM7.6
- removed D1: LED, LED_SMD:LED_1210_3225Metric_Pad1.42x2.65mm_HandSolder
- removed DISP1_CONN1: DISPLAY_CONNECTOR, Connector_JST:JST_PH_S7B-PH-K_1x07_P2.00mm_Horizontal
- removed H5, H6: MountingHole_Pad, MountingHole:MountingHole_2.2mm_M2_Pad
- removed J3: Conn_01x06_Pin, Connector_PinHeader_2.54mm:PinHeader_1x06_P2.54mm_Horizontal
- removed R1: R_330, Resistor_THT:R_Axial_DIN0204_L3.6mm_D1.6mm_P5.08mm_Horizontal
- removed REF**: MountingHole_2.2mm_M2, MountingHole:MountingHole_2.2mm_M2
- added AUDIO1: AUDIO, vgc-zero-footprints:Untitled, B.Cu at (73.3, 51.7)
- J1: value Conn_01x06_Pin -> Conn_02x06_Top_Bottom; footprint Connector_PinHeader_2.54mm:PinHeader_1x06_P2.54mm_Horizontal -> Connector_PinSocket_2.54mm:PinSocket_2x05_P2.54mm_Horizontal
- J2: value Conn_01x06_Pin -> Conn_01x03_Socket; footprint Connector_PinHeader_2.54mm:PinHeader_1x06_P2.54mm_Horizontal -> Connector_JST:JST_SH_SM03B-SRSS-TB_1x03-1MP_P1.00mm_Horizontal
- MCU1: footprint Module:RaspberryPi_Pico_Common_THT -> Module:RaspberryPi_Pico_Common_Unspecified
- SW11: value SW_SPDT -> SW_Push; footprint Button_Switch_THT:SW_Slide_SPDT_Angled_CK_OS102011MA1Q -> Button_Switch_THT:SW_Tactile_SPST_Angled_PTS645Vx58-2LFS
- moved SW11 54.4 mm to (70.3, 40.7), turned to 180 degrees
- moved J1 28.3 mm to (85.1, 115.3), turned to 90 degrees
- moved MCU1 24.1 mm to (85.1, 63.5)
- moved J2 22.8 mm to (77.0, 95.0), turned to 180 degrees
- moved SW2 5.25 mm to (103.0, 104.2)
- moved SW3 5.25 mm to (98.2, 94.2)
- moved SW4 5.25 mm to (93.5, 108.8)
- moved SW5 5.25 mm to (88.8, 98.8)
- moved SW6 5.25 mm to (77.5, 103.7)
- moved SW7 5.25 mm to (70.0, 117.7)
- moved SW8 5.25 mm to (70.0, 100.7)
- moved SW9 5.25 mm to (56.0, 110.2)
- moved SW10 2.46 mm to (61.5, 82.5), turned to -90 degrees
- moved SW1 2.14 mm to (102.2, 82.8), turned to -90 degrees
Connections:
- net Net-(MCU1-GPIO10) renamed /GPIO10
- net Net-(MCU1-GPIO11) renamed /GPIO11
- net Net-(MCU1-GPIO2) renamed /GPIO2
- net Net-(MCU1-GPIO3) renamed /GPIO3
- net Net-(MCU1-GPIO4) renamed /GPIO4
- net Net-(MCU1-GPIO5) renamed /GPIO5
- net Net-(MCU1-GPIO6) renamed /GPIO6
- net Net-(MCU1-GPIO7) renamed /GPIO7
- net Net-(MCU1-GPIO8) renamed /GPIO8
- net Net-(MCU1-GPIO9) renamed /GPIO9
- DISP1 pad 1: /GND -> +3.3V
- J1 pad 1: Net-(J1-Pin_1) -> +3.3V
- J1 pad 2: Net-(J1-Pin_2) -> /EN
- J1 pad 3: Net-(J1-Pin_3) -> /3V3_EN
- J1 pad 4: Net-(J1-Pin_4) -> /GPIO0
- J1 pad 5: Net-(J1-Pin_5) -> /GPIO1
- J1 pad 6: 3V3 -> GND
- J2 pad 1: /GND -> /SWCLK
- J2 pad 2: Net-(J2-Pin_2) -> /SWDIO
- J2 pad 3: Net-(J2-Pin_3) -> GND
- MCU1 pad 1: Net-(J2-Pin_4) -> /GPIO0
- MCU1 pad 13: /GND -> GND
- MCU1 pad 16: Net-(J3-Pin_5) -> /GPIO12
- MCU1 pad 17: Net-(J3-Pin_4) -> /GPIO13
- MCU1 pad 18: /GND -> GND
- MCU1 pad 19: Net-(J3-Pin_3) -> /GPIO14
- MCU1 pad 2: Net-(J2-Pin_5) -> /GPIO1
- MCU1 pad 20: Net-(J3-Pin_2) -> /GPIO15
- MCU1 pad 21: Net-(MCU1-GPIO16) -> /GPIO16
- MCU1 pad 23: /GND -> GND
- MCU1 pad 28: /GND -> GND
- MCU1 pad 29: Net-(Buzz1-+) -> /GPIO22
- MCU1 pad 3: /GND -> GND
- MCU1 pad 30: Net-(J2-Pin_2) -> /EN
- MCU1 pad 31: Net-(J1-Pin_4) -> /GPIO26
- MCU1 pad 32: Net-(J1-Pin_3) -> /GPIO27
- MCU1 pad 33: Net-(J1-Pin_1) -> /AGND
- MCU1 pad 34: Net-(J1-Pin_2) -> /GPIO28
- MCU1 pad 35: Net-(J1-Pin_5) -> /ADC_VREF
- MCU1 pad 36: 3V3 -> +3.3V
- MCU1 pad 37: Net-(J2-Pin_3) -> /3V3_EN
- MCU1 pad 38: /GND -> GND
- MCU1 pad 8: /GND -> GND
- SW1 pad 1: /GND -> GND
- SW10 pad 1: /GND -> GND
- SW11 pad 1: /GND -> GND
- SW11 pad 2: Net-(J2-Pin_3) -> /GPIO12
- SW2 pad 1: /GND -> GND
- SW3 pad 1: /GND -> GND
- SW4 pad 1: /GND -> GND
- SW5 pad 1: /GND -> GND
- SW6 pad 1: /GND -> GND
- SW7 pad 1: /GND -> GND
- SW8 pad 1: /GND -> GND
- SW9 pad 1: /GND -> GND
Routing:
- net 3V3: track 132.9 -> 0.00 mm
- net Net-(J2-Pin_3): track 107.9 -> 0.00 mm
- net Net-(J1-Pin_5): track 88.1 -> 0.00 mm
- net Net-(J2-Pin_4): track 81.1 -> 0.00 mm
- net Net-(J2-Pin_5): track 79.2 -> 0.00 mm
- net Net-(J1-Pin_1): track 70.3 -> 0.00 mm
- net Net-(J1-Pin_2): track 68.2 -> 0.00 mm
- net /GPIO8: track 66.1 -> 0.00 mm
- net /GPIO10: track 62.3 -> 0.00 mm
- net Net-(J1-Pin_3): track 61.3 -> 0.00 mm
- net Net-(MCU1-GPIO16): track 61.3 -> 0.00 mm
- net /GPIO3: track 59.9 -> 0.00 mm
- net /GPIO7: track 58.3 -> 0.00 mm
- net /GPIO5: track 57.8 -> 0.00 mm
- net Net-(J1-Pin_4): track 57.6 -> 0.00 mm
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- added copper zone on F.Cu, net +3.3V
- removed copper zone on F.Cu, net /GND
Other:
- outline, holes or cut-outs redrawn
- board text added: "S022026"
- board text added: "vgc zero v1.2.0"
- board text removed: "RoHS"
- board text removed: "S012026"
- board text removed: "vgc zero v1.1.4"
